Commit message: 第二次提交

File: original_isaacgym/python/examples/resources/tinker/model_dir/urdf/tinker_urdf_inv1.urdf (robot description, URDF)
Before this commit: robot tinker_urdf, 11 links, 10 joints
Links:
- link link_l_ankle: geometry collision cylinder length=0.13 radius=0.01; collision mesh filename=../meshes/link_l_ankle.STL
- link link_r_ankle: geometry collision cylinder length=0.13 radius=0.015; collision mesh filename=../meshes/link_r_ankle.STL

File: original_isaacgym/python/examples/resources/tinker/urdf/tinker_urdf_inv1.urdf (robot description, URDF)
Before this commit: robot tinker_urdf, 11 links, 10 joints
Links:
- link link_l_ankle: geometry collision cylinder length=0.13 radius=0.01; collision mesh filename=../meshes/link_l_ankle.STL
- link link_r_ankle: geometry collision cylinder length=0.13 radius=0.015; collision mesh filename=../meshes/link_r_ankle.STL

Commit message: 第四次提交

File: original_isaacgym/python/examples/resources/tinker/model_dir/urdf/tinker_urdf_inv1.urdf (robot description, URDF)
Before this commit: robot tinker_urdf, 11 links, 10 joints
Links:
- link link_l_ankle: geometry collision mesh filename=../meshes/link_l_ankle.STL; visual mesh filename=../meshes/link_l_ankle.STL
- link link_r_ankle: geometry collision mesh filename=../meshes/link_r_ankle.STL; visual mesh filename=../meshes/link_r_ankle.STL
